File: Power_supply_PCB_Design.kicad_sch (KiCad schematic)
At the start: 17 parts, among them J1 Conn_01x02_Pin, J2 Conn_01x02_Pin, J3 Conn_01x03_Pin, J4 Conn_01x03_Pin, J5 Screw_Terminal_01x02, J6 Barrel_Jack_Switch, J7 Screw_Terminal_01x02, SW1 SW_Wuerth_450301014042, U1 LM7805_TO220, U2 LM317_TO-220

Commit message: Additional Bug Fixes
Other:
- note added: "Input and 5V Circuit"
- note removed: "Input amd 5V Circuit"
Changed lines of the file:
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@@
 		)
 	)
-	(text "Input amd 5V Circuit"
+	(text "Input and 5V Circuit"
 		(exclude_from_sim no)
 		(at 35.56 15.24 0)
